Commit message: merged dd490cd

File: vrx_description/configs/default_config.urdf (robot description, URDF)
Before this commit: robot WAM-V, 23 links, 22 joints
Links:
- removed link front_left_camera_link
- removed link front_left_camera_post_arm_link
- removed link front_left_camera_post_link
- removed link front_right_camera_link
- removed link front_right_camera_post_arm_link
- removed link front_right_camera_post_link
- removed link middle_right_camera_link
- removed link middle_right_camera_post_arm_link
- removed link middle_right_camera_post_link
- added link left_camera_link, mass 0.3; collision box size=0.036 0.03 0.03; collision cylinder length=0.042 radius=0.015
- added link left_camera_post_arm_link, mass 0.1; collision cylinder length=0.065 radius=0.008; visual mesh filename=package://vrx_gazebo/models/sensor_post/mesh/sensor_post_ar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
- added link left_camera_post_link, mass 0.15885; collision cylinder length=0.1765 radius=0.0076; visual cylinder length=0.1765 radius=0.0076
- added link middle_camera_link, mass 0.3; collision box size=0.036 0.03 0.03; collision cylinder length=0.042 radius=0.015
- added link middle_camera_post_arm_link, mass 0.1; collision cylinder length=0.065 radius=0.008; visual mesh filename=package://vrx_gazebo/models/sensor_post/mesh/sensor_post_ar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
- added link middle_camera_post_link, mass 0.15885; collision cylinder length=0.1765 radius=0.0076; visual cylinder length=0.1765 radius=0.0076
- added link right_camera_link, mass 0.3; collision box size=0.036 0.03 0.03; collision cylinder length=0.042 radius=0.015
- added link right_camera_post_arm_link, mass 0.1; collision cylinder length=0.065 radius=0.008; visual mesh filename=package://vrx_gazebo/models/sensor_post/mesh/sensor_post_ar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
- added link right_camera_post_link, mass 0.15885; collision cylinder length=0.1765 radius=0.0076; visual cylinder length=0.1765 radius=0.0076
Joints:
- removed joint base_to_front_left_camera_post_joint
- removed joint base_to_front_right_camera_post_joint
- removed joint base_to_middle_right_camera_post_joint
- removed joint front_left_camera_post_arm_to_front_left_camera_joint
- removed joint front_left_camera_post_to_front_left_camera_post_arm_joint
- removed joint front_right_camera_post_arm_to_front_right_camera_joint
- removed joint front_right_camera_post_to_front_right_camera_post_arm_joint
- removed joint middle_right_camera_post_arm_to_middle_right_camera_joint
- removed joint middle_right_camera_post_to_middle_right_camera_post_arm_joint
- added joint base_to_left_camera_post_joint: type fixed, parent base_link, child left_camera_post_link, origin xyz=0.7 0.1 1.38475 rpy=0 0 0
- added joint base_to_middle_camera_post_joint: type fixed, parent base_link, child middle_camera_post_link, origin xyz=0.7 0.0 1.38475 rpy=0 0 0
- added joint base_to_right_camera_post_joint: type fixed, parent base_link, child right_camera_post_link, origin xyz=0.7 -0.1 1.38475 rpy=0 0 0
- added joint left_camera_post_arm_to_left_camera_joint: type fixed, parent left_camera_post_arm_link, child left_camera_link, origin xyz=0.02 0 0.027 rpy=0 0 0.523598775598
- added joint left_camera_post_to_left_camera_post_arm_joint: type fixed, parent left_camera_post_link, child left_camera_post_arm_link, origin xyz=0.03 0 0.08825 rpy=0 0 0
- added joint middle_camera_post_arm_to_middle_camera_joint: type fixed, parent middle_camera_post_arm_link, child middle_camera_link, origin xyz=0.02 0 0.027 rpy=0 0 0.0
- added joint middle_camera_post_to_middle_camera_post_arm_joint: type fixed, parent middle_camera_post_link, child middle_camera_post_arm_link, origin xyz=0.03 0 0.08825 rpy=0 0 0
- added joint right_camera_post_arm_to_right_camera_joint: type fixed, parent right_camera_post_arm_link, child right_camera_link, origin xyz=0.02 0 0.027 rpy=0 0 -0.523598775598
- added joint right_camera_post_to_right_camera_post_arm_joint: type fixed, parent right_camera_post_link, child right_camera_post_arm_link, origin xyz=0.03 0 0.08825 rpy=0 0 0

Commit message: change camera configuration

File: vrx_description/configs/default_config.urdf (robot description, URDF)
Before this commit: robot WAM-V, 22 links, 21 joints
Links:
- removed link front_left_camera_link
- removed link front_left_camera_post_arm_link
- removed link front_left_camera_post_link
- removed link front_right_camera_link
- removed link front_right_camera_post_arm_link
- removed link front_right_camera_post_link
- removed link middle_right_camera_link
- removed link middle_right_camera_post_arm_link
- removed link middle_right_camera_post_link
- added link cpu_cases_link, mass 20; collision box size=0.375 0.64 0.28; collision box size=0.595 0.83 0.47
- added link left_camera_link, mass 0.3; collision box size=0.036 0.03 0.03; collision cylinder length=0.042 radius=0.015
- added link left_camera_post_arm_link, mass 0.1; collision cylinder length=0.065 radius=0.008; visual mesh filename=package://vrx_gazebo/models/sensor_post/mesh/sensor_post_ar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
- added link left_camera_post_link, mass 0.15885; collision cylinder length=0.1765 radius=0.0076; visual cylinder length=0.1765 radius=0.0076
- added link middle_camera_link, mass 0.3; collision box size=0.036 0.03 0.03; collision cylinder length=0.042 radius=0.015
- added link middle_camera_post_arm_link, mass 0.1; collision cylinder length=0.065 radius=0.008; visual mesh filename=package://vrx_gazebo/models/sensor_post/mesh/sensor_post_ar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
- added link middle_camera_post_link, mass 0.15885; collision cylinder length=0.1765 radius=0.0076; visual cylinder length=0.1765 radius=0.0076
- added link right_camera_link, mass 0.3; collision box size=0.036 0.03 0.03; collision cylinder length=0.042 radius=0.015
- added link right_camera_post_arm_link, mass 0.1; collision cylinder length=0.065 radius=0.008; visual mesh filename=package://vrx_gazebo/models/sensor_post/mesh/sensor_post_ar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
- added link right_camera_post_link, mass 0.15885; collision cylinder length=0.1765 radius=0.0076; visual cylinder length=0.1765 radius=0.0076
- link dummy_link: geometry collision box size=0.65 0.2 0.1; collision box size=0.65 0.2 0.1
- link gps_wamv_link: geometry collision cylinder length=0.05 radius=0.015; collision cylinder length=0.1 radius=0.15
- link left_engine_link: geometry collision box size=0.12 0.15 0.12; collision box size=0.2 0.15 0.83
- link left_propeller_link: geometry collision cylinder length=0.18 radius=0.24; visual mesh filename=package://wamv_description/models/propeller/mesh/propeller.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
- link right_engine_link: geometry collision box size=0.12 0.15 0.12; collision box size=0.2 0.15 0.83
- link right_propeller_link: geometry collision cylinder length=0.18 radius=0.24; visual mesh filename=package://wamv_description/models/propeller/mesh/propeller.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
Joints:
- removed joint base_to_front_left_camera_post_joint
- removed joint base_to_front_right_camera_post_joint
- removed joint base_to_middle_right_camera_post_joint
- removed joint front_left_camera_post_arm_to_front_left_camera_joint
- removed joint front_left_camera_post_to_front_left_camera_post_arm_joint
- removed joint front_right_camera_post_arm_to_front_right_camera_joint
- removed joint front_right_camera_post_to_front_right_camera_post_arm_joint
- removed joint middle_right_camera_post_arm_to_middle_right_camera_joint
- removed joint middle_right_camera_post_to_middle_right_camera_post_arm_joint
- added joint base_to_left_camera_post_joint: type fixed, parent base_link, child left_camera_post_link, origin xyz=0.7 0.1 1.38475 rpy=0 0 0
- added joint base_to_middle_camera_post_joint: type fixed, parent base_link, child middle_camera_post_link, origin xyz=0.7 0.0 1.38475 rpy=0 0 0
- added joint base_to_right_camera_post_joint: type fixed, parent base_link, child right_camera_post_link, origin xyz=0.7 -0.1 1.38475 rpy=0 0 0
- added joint chasis_cpu_cases_joint: type fixed, parent base_link, child cpu_cases_link, origin xyz=-0.15 0 1.53 rpy=0 0 0
- added joint left_camera_post_arm_to_left_camera_joint: type fixed, parent left_camera_post_arm_link, child left_camera_link, origin xyz=0.02 0 0.027 rpy=0 0 0.523598775598
- added joint left_camera_post_to_left_camera_post_arm_joint: type fixed, parent left_camera_post_link, child left_camera_post_arm_link, origin xyz=0.03 0 0.08825 rpy=0 0 0
- added joint middle_camera_post_arm_to_middle_camera_joint: type fixed, parent middle_camera_post_arm_link, child middle_camera_link, origin xyz=0.02 0 0.027 rpy=0 0 0.0
- added joint middle_camera_post_to_middle_camera_post_arm_joint: type fixed, parent middle_camera_post_link, child middle_camera_post_arm_link, origin xyz=0.03 0 0.08825 rpy=0 0 0
- added joint right_camera_post_arm_to_right_camera_joint: type fixed, parent right_camera_post_arm_link, child right_camera_link, origin xyz=0.02 0 0.027 rpy=0 0 -0.523598775598
- added joint right_camera_post_to_right_camera_post_arm_joint: type fixed, parent right_camera_post_link, child right_camera_post_arm_link, origin xyz=0.03 0 0.08825 rpy=0 0 0

File: vrx_description/configs/sensor_config.xacro (robot description, xacro)
@@ -9,7 +9,7 @@
       <xacro:wamv_p3d name="p3d_wamv" />
     <!-- === wamv_camera === -->
-      <xacro:wamv_camera y="0.1" x="0.75" name="front_left_camera" P="${radians(15)}" />
-      <xacro:wamv_camera y="-0.1" x="0.75" name="front_right_camera" P="${radians(15)}" />
-      <xacro:wamv_camera y="0.3" x="0.75" name="middle_right_camera" P="${radians(15)}" />
+      <xacro:wamv_camera y="0.1" x="0.75" Y="${radians(30)}" name="left_camera" />
+      <xacro:wamv_camera y="-0.1" x="0.75" Y="${radians(-30)}" name="right_camera" />
+      <xacro:wamv_camera y="0" x="0.75" Y="${radians(0)}" name="middle_camera" />
     <!-- === lidar === -->
       <xacro:lidar P="${radians(8)}" type="16_beam" name="lidar_wamv" />

Commit message: Fixed issue #3 by rebuilding the urdf and grouping the namespace to wamv

File: vrx_description/configs/default_config.urdf (robot description, URDF)
Before this commit: robot WAM-V, 22 links, 21 joints
Links:
- added link cpu_cases_link, mass 20; collision box size=0.375 0.64 0.28; collision box size=0.595 0.83 0.47
- link dummy_link: geometry collision box size=0.65 0.2 0.1; collision box size=0.65 0.2 0.1
- link gps_wamv_link: geometry collision cylinder length=0.05 radius=0.015; collision cylinder length=0.1 radius=0.15
- link left_engine_link: geometry collision box size=0.12 0.15 0.12; collision box size=0.2 0.15 0.83
- link left_propeller_link: geometry collision cylinder length=0.18 radius=0.24; visual mesh filename=package://wamv_description/models/propeller/mesh/propeller.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
- link right_engine_link: geometry collision box size=0.12 0.15 0.12; collision box size=0.2 0.15 0.83
- link right_propeller_link: geometry collision cylinder length=0.18 radius=0.24; visual mesh filename=package://wamv_description/models/propeller/mesh/propeller.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
Joints:
- added joint chasis_cpu_cases_joint: type fixed, parent base_link, child cpu_cases_link, origin xyz=-0.15 0 1.53 rpy=0 0 0

File: vrx_description/configs/thruster_config.xacro (robot description, xacro)
@@ -8,4 +8,5 @@
     <plugin name="wamv_gazebo_thrust" filename="libusv_gazebo_thrust_plugin.so">
       <cmdTimeout>1.0</cmdTimeout>
+      <robotNamespace>${namespace}</robotNamespace>
       <xacro:include filename="$(find wamv_gazebo)/urdf/thruster_layouts/wamv_gazebo_thruster_config.xacro" />
         <xacro:wamv_gazebo_thruster_config name="left" />
