Commit message: Multiple changes in this one: Fixed up name spaces so that all developed nodes are working.

File: vrx_description/configs/sensor_config.xacro (robot description, xacro)
@@ -13,5 +13,5 @@
       <xacro:wamv_camera y="0" x="0.75" Y="${radians(0)}" name="middle_camera" />
     <!-- === lidar === -->
-      <xacro:lidar P="${radians(8)}" type="16_beam" name="lidar_wamv" />
+      <xacro:lidar P="0" type="16_beam" name="lidar_wamv" />
   </xacro:macro>
 </robot>

File: vrx_description/configs/usyd_wamv.urdf (robot description, URDF)
Before this commit: robot WAM-V, 25 links, 24 joints
Joints:
- joint lidar_wamv_post_arm_to_lidar_wamv_joint: origin xyz=0.04 0 0.05 rpy=0 0.13962634016 0 -> xyz=0.04 0 0.05 rpy=0 0 0
